Commit message: 1227 commit

File: urdf/aimibot.urdf (robot description, URDF)
Before this commit: robot aimibot, 5 links, 4 joints
Links:
- link base_link: geometry collision mesh filename=package://aimibot_description/meshes/base_link.STL; visual mesh filename=package://aimibot_description/meshes/base_link.STL
- link laser_link: geometry collision mesh filename=package://aimibot_description/meshes/laser_link.STL; visual mesh filename=package://aimibot_description/meshes/laser_link.STL
- link wheel_left_link: geometry collision mesh filename=package://aimibot_description/meshes/wheel_left_link.STL; visual mesh filename=package://aimibot_description/meshes/wheel_left_link.STL
- link wheel_right_link: geometry collision mesh filename=package://aimibot_description/meshes/wheel_right_link.STL; visual mesh filename=package://aimibot_description/meshes/wheel_right_link.STL
